Commit message: improve urdf/scan filter

File: src/sweeper_bot/src/description/sick.xacro (robot description, xacro)
@@ -22,7 +22,7 @@
     </link>
     <joint name="sick_joint" type="fixed">
-        <parent link="chassis"/>
+        <parent link="base_link"/>
         <child link="sick_link"/>
-        <origin xyz="${chassis_length} 0 ${chassis_height/3}" rpy="0 0 0"/>
+        <origin xyz=".813 0 .127" rpy="0 0 0"/>
     </joint>
     <link name="sick_lidar_frame"/>

Commit message: localization improvements

File: src/sweeper_bot/src/description/sick.xacro (robot description, xacro)
@@ -27,5 +27,5 @@
     </joint>
     <link name="sick_lidar_frame"/>
-    <joint name="sick_lidar_frame" type="fixed">
+    <joint name="sick_frame_joint" type="fixed">
         <origin xyz="0 0 0" rpy="0 0 0"/>
         <parent link="sick_link"/>
